File: Hardware/Electric Layout/Power_control.kicad_pcb (KiCad board)
At the start: 2 copper layers, 60 x 80 mm, 22 parts, among them J2 Power IN, J3 CAN BUS Modul, J4 CAN Connect, J5 To USB, Q1 IRF9540N, Q2 2N3904

Commit message: Add files via upload
New layout
Parts:
- J5: value To USB -> To USB converter
- RN1: value Pull Up 47k -> Pull Up 10k
- moved D1 1.12 mm to (65.0, 67.8)
Connections:
- ESP1 pad 3: Green Pin 22 (coolant) -> Net-(ESP1-SENSOR_VP/GPIO36/ADC1_CH0)
- ESP1 pad 4: directly from Oil LED -> /Volt Measurement
- ESP1 pad 7: /Volt Measurement -> Net-(ESP1-32K_XP/GPIO32/ADC1_CH4)
- ESP32_1 pad 13: /Volt Measurement -> Net-(ESP1-32K_XP/GPIO32/ADC1_CH4)
- ESP32_1 pad 16: directly from Oil LED -> /Volt Measurement
- ESP32_1 pad 17: Green Pin 22 (coolant) -> Net-(ESP1-SENSOR_VP/GPIO36/ADC1_CH0)
- RN1 pad 2: Green Pin 22 (coolant) -> unconnected-(RN1-R1-Pad2)
- RN1 pad 3: directly from Oil LED -> Net-(ESP1-SENSOR_VP/GPIO36/ADC1_CH0)
Routing:
- net directly from Oil LED: track 11.1 -> 0.00 mm
- net /Volt Measurement: track 205.5 -> 194.6 mm
- net Green Pin 22 (coolant): track 10.9 -> 0.00 mm
- net Net-(ESP1-SENSOR_VP/GPIO36/ADC1_CH0): track 0.00 -> 9.30 mm
- net Net-(ESP1-32K_XP/GPIO32/ADC1_CH4): track 0.00 -> 3.50 mm
- net Net-(D1-K): track 23.5 -> 24.6 mm
- net /Stay On: track 206.2 -> 207.1 mm
- net GND: track 345.5 -> 344.7 mm
