File: Hardware/KICAD/BrakeOutBoard.kicad_pcb (KiCad board)
At the start: 2 copper layers, 63 x 80 mm, 64 parts, among them J20 Conn_01x19_Socket, J5 Conn_01x19_Socket, K15 K15, K30 K30, K31 K31, Q1 MMDT3904, Q2 LBSS84LT1G, U1 LTV-847, U101 SN65HVD230DR, U2 LTV-847, U3 LVT 817, U4 LTV-847, U501 MCP23017_ML

Commit message: Add files via upload
Parts:
- added ESP1: ~, PCM_Espressif:ESP32-DevKitC, F.Cu at (183.5, 123.9)
- added K501: K31, Connector_Wire:SolderWire-0.5sqmm_1x01_D0.9mm_OD2.1mm, F.Cu at (136.5, 106.6)
- added K502: K31, Connector_Wire:SolderWire-0.5sqmm_1x01_D0.9mm_OD2.1mm, F.Cu at (132.7, 106.6)
- added K503: K31, Connector_Wire:SolderWire-0.5sqmm_1x01_D0.9mm_OD2.1mm, F.Cu at (132.7, 99.2)
- added K504: K31, Connector_Wire:SolderWire-0.5sqmm_1x01_D0.9mm_OD2.1mm, F.Cu at (136.5, 99.2)
- U501: footprint Package_DFN_QFN:QFN-28-1EP_6x6mm_P0.65mm_EP4.25x4.25mm -> Package_SO:SSOP-28_5.3x10.2mm_P0.65mm
- moved J20 45.7 mm to (137.7, 149.2), turned to 90 degrees
- moved R301 9.80 mm to (139.2, 89.5), turned to 0 degrees
- moved R502 4.10 mm to (156.8, 118.3), turned to 180 degrees
- moved U501 2.84 mm to (146.6, 112.4), turned to 0 degrees
- moved C501 2.39 mm to (149.4, 121.3), turned to 0 degrees
- moved C502 2.04 mm to (154.7, 115.2)
- moved R501 2.03 mm to (158.1, 115.0)
- moved R503 0.26 mm to (149.7, 120.0)
Connections:
- J20 pad 1: GND -> unconnected-(J20-Pin_1-Pad1)
- J20 pad 11: GPIO 17 (PIN 28) -> Net-(J20-Pin_11)
- J20 pad 12: GPIO 16 (PIN 27) -> GPIO 19 (PIN 31)
- J20 pad 13: GPIO 4 (PIN 26) -> GND
- J20 pad 14: GPIO 0 (PIN 25) -> CAN Modul RTX
- J20 pad 15: Net-(J20-Pin_15) -> unconnected-(J20-Pin_15-Pad15)
- J20 pad 17: unconnected-(J20-Pin_17-Pad17) -> CAN Modul CTX
- J20 pad 18: unconnected-(J20-Pin_18-Pad18) -> Net-(J20-Pin_18)
- J20 pad 19: unconnected-(J20-Pin_19-Pad19) -> GND
- J20 pad 2: Net-(J20-Pin_2) -> unconnected-(J20-Pin_2-Pad2)
- J20 pad 3: CAN Modul CTX -> unconnected-(J20-Pin_3-Pad3)
- J20 pad 5: unconnected-(J20-Pin_5-Pad5) -> Net-(J20-Pin_5)
- J20 pad 6: CAN Modul RTX -> GPIO 0 (PIN 25)
- J20 pad 7: GND -> GPIO 4 (PIN 26)
- J20 pad 8: GPIO 19 (PIN 31) -> GPIO 16 (PIN 27)
- J20 pad 9: Net-(J20-Pin_9) -> GPIO 17 (PIN 28)
- MOSi_1 pad 1: Net-(J20-Pin_2) -> Net-(J20-Pin_18)
- R10 pad 5: PortExpander GPA2 -> GPIO 4 (PIN 26)
- R10 pad 6: PortExpander GPA3 -> PortExpander GPA2
- R13 pad 5: PortExpander GPB5 -> PortExpander GPB3
- R13 pad 6: PortExpander GPB4 -> PortExpander GPB2
- R13 pad 7: PortExpander GPB3 -> PortExpander GPB1
- R13 pad 8: PortExpander GPB2 -> PortExpander GPB0
- R9 pad 5: PortExpander GPB1 -> GPIO 14 (PIN 12)
- R9 pad 6: PortExpander GPB0 -> GPIO 13 (PIN 15)
- R9 pad 7: PortExpander GPA5 -> PortExpander GPA4
- R9 pad 8: PortExpander GPA4 -> PortExpander GPA3
- SLK_1 pad 1: Net-(J20-Pin_9) -> Net-(J20-Pin_11)
- TFT_DC_1 pad 1: Net-(J20-Pin_15) -> Net-(J20-Pin_5)
- U1 pad 11: PortExpander GPA3 -> PortExpander GPA2
- U1 pad 9: PortExpander GPA2 -> GPIO 4 (PIN 26)
- U2 pad 11: PortExpander GPB0 -> GPIO 13 (PIN 15)
- U2 pad 13: PortExpander GPA5 -> PortExpander GPA4
- U2 pad 15: PortExpander GPA4 -> PortExpander GPA3
- U2 pad 9: PortExpander GPB1 -> GPIO 14 (PIN 12)
- U4 pad 11: PortExpander GPB4 -> PortExpander GPB2
- U4 pad 13: PortExpander GPB3 -> PortExpander GPB1
- U4 pad 15: PortExpander GPB2 -> PortExpander GPB0
- U4 pad 9: PortExpander GPB5 -> PortExpander GPB3
- U501 pad 1: PortExpander GPB4 -> PortExpander GPB0
- U501 pad 10: unconnected-(U501-NC-Pad10) -> GND
- U501 pad 11: GND -> unconnected-(U501-NC-Pad11)
- U501 pad 12: GND -> GPIO 27 (PIN 11)
- U501 pad 13: GND -> GPIO 26 (PIN 10)
- U501 pad 14: Net-(U501-~{RESET}) -> unconnected-(U501-NC-Pad14)
- U501 pad 15: GPIO 32 (PIN 7) -> GND
- U501 pad 16: GPIO 33 (PIN 8) -> GND
- U501 pad 17: PortExpander GPA0 -> GND
- U501 pad 18: PortExpander GPA1 -> Net-(U501-~{RESET})
- U501 pad 19: PortExpander GPA2 -> GPIO 32 (PIN 7)
- U501 pad 2: PortExpander GPB5 -> PortExpander GPB1
- U501 pad 20: PortExpander GPA3 -> GPIO 33 (PIN 8)
- U501 pad 21: PortExpander GPA4 -> PortExpander GPA0
- U501 pad 22: PortExpander GPA5 -> PortExpander GPA1
- U501 pad 23: unconnected-(U501-GPA6-Pad23) -> PortExpander GPA2
- U501 pad 24: unconnected-(U501-GPA7-Pad24) -> PortExpander GPA3
- U501 pad 25: PortExpander GPB0 -> PortExpander GPA4
- U501 pad 26: PortExpander GPB1 -> PortExpander GPA5
- U501 pad 27: PortExpander GPB2 -> /Port Expander/GPA6
- U501 pad 28: PortExpander GPB3 -> /Port Expander/GPA7
- U501 pad 3: unconnected-(U501-GPB6-Pad3) -> PortExpander GPB2
- U501 pad 4: unconnected-(U501-GPB7-Pad4) -> PortExpander GPB3
- U501 pad 5: 3,3 V from ESP -> PortExpander GPB4
- U501 pad 6: GND -> PortExpander GPB5
- U501 pad 7: unconnected-(U501-NC-Pad7) -> /Port Expander/GPB6
- U501 pad 8: GPIO 27 (PIN 11) -> /Port Expander/GPB7
- U501 pad 9: GPIO 26 (PIN 10) -> 3,3 V from ESP
Routing:
- net GPIO 4 (PIN 26): track 0.00 -> 197.2 mm
- net GPIO 14 (PIN 12): track 0.00 -> 118.6 mm
- net GPIO 13 (PIN 15): track 0.00 -> 117.1 mm
- net PortExpander GPB5: track 86.3 -> 0.00 mm, vias 1 -> 0
- net PortExpander GPB4: track 85.9 -> 0.00 mm, vias 1 -> 0
- net PortExpander GPB1: track 42.1 -> 96.0 mm, vias 0 -> 2
- net PortExpander GPB0: track 42.0 -> 81.1 mm
- net PortExpander GPA5: track 38.5 -> 0.00 mm
- net 3,3 V from ESP: track 265.7 -> 290.7 mm, vias 2 -> 0
- net /Port Expander/GPA6: track 0.00 -> 24.3 mm, vias 0 -> 1
- net PortExpander GPA3: track 59.7 -> 35.7 mm
- net /Port Expander/GPA7: track 0.00 -> 20.8 mm, vias 0 -> 1
- net PortExpander GPB3: track 94.4 -> 76.2 mm, vias 2 -> 1
- net K15: track 102.1 -> 117.4 mm
- net PortExpander GPB2: track 90.2 -> 76.9 mm, vias 0 -> 1
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