File: Hardware/KICAD/BrakeOutBoard.kicad_sch (KiCad schematic)
At the start: 11 parts, among them J20 Conn_01x19_Socket, J5 Conn_01x19_Socket

Commit message: Add files via upload
Connections:
- net CAN Modul CTX: now also J20.17 (Pin_17); no longer J20.3 (Pin_3)
- net CAN Modul RTX: now also J20.14 (Pin_14); no longer J20.6 (Pin_6)
- net GND: now also J20.13 (Pin_13), J20.19 (Pin_19); no longer J20.1 (Pin_1), J20.7 (Pin_7)
- net GPIO 0 (PIN 25): now also J20.6 (Pin_6); no longer J20.14 (Pin_14)
- net GPIO 16 (PIN 27): now also J20.8 (Pin_8); no longer J20.12 (Pin_12)
- net GPIO 17 (PIN 28): now also J20.9 (Pin_9); no longer J20.11 (Pin_11)
- net GPIO 19 (PIN 31): now also J20.12 (Pin_12); no longer J20.8 (Pin_8)
- net GPIO 4 (PIN 26): now also J20.7 (Pin_7); no longer J20.13 (Pin_13)
- net at J20.15 (Pin_15): no longer TFT_DC_1.1 (Pin_1)
- net at J20.18 (Pin_18): now also MOSi_1.1 (Pin_1)
- net at J20.2 (Pin_2): no longer MOSi_1.1 (Pin_1)
- net at J20.5 (Pin_5): now also TFT_DC_1.1 (Pin_1)
- net at SLK_1.1 (Pin_1): now also J20.11 (Pin_11); no longer J20.9 (Pin_9)
Other:
- moved on the sheet: J20
Changed lines of the file:
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@@
 	(symbol
 		(lib_id "Connector:Conn_01x19_Socket")
-		(at 186.69 88.9 0)
-		(mirror y)
+		(at 186.69 88.9 180)
 		(unit 1)
 		(exclude_from_sim no)
@@
 		(dnp no)
 		(property "Reference" "J20"
-			(at 189.484 61.468 0)
+			(at 189.484 116.332 0)
 			(effects
 				(font
@@
 		)
 		(property "Value" "Conn_01x19_Socket"
-			(at 187.325 114.3 0)
+			(at 187.325 63.5 0)
 			(effects
 				(font
