File: Hardware/KICAD/Latch_Circuit.kicad_sch (KiCad schematic)
At the start: 14 parts, among them K15 K15, K30 K30, K31 K31, Q1 MMDT3904, Q2 LBSS84LT1G

Commit message: Add files via upload
Changed lines of the file:
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@@
 	)
 	(global_label "StayOn"
-		(shape input)
+		(shape output)
 		(at 234.95 95.25 0)
 		(fields_autoplaced yes)
@@
 	)
 	(global_label "VoltMeasurement"
-		(shape input)
+		(shape output)
 		(at 194.31 118.11 0)
 		(fields_autoplaced yes)
