File: Hardware/KICAD/Optocopler.kicad_sch (KiCad schematic)
At the start: 24 parts, among them U1 LTV-847, U2 LTV-847, U3 LVT 817, U4 LTV-847

Commit message: Add files via upload
Connections:
- net PortExpander GPA5 is gone; now on net PortExpander GPA4: R9.7, U2.13
- net PortExpander GPB4 is gone; now on net PortExpander GPB2: R13.6, U4.11
- net PortExpander GPB5 is gone; now on net PortExpander GPB3: R13.5, U4.9
- net PortExpander GPA2: now also R10.6, U1.11; no longer R10.5, U1.9
- net PortExpander GPA3: now also R9.8, U2.15; no longer R10.6, U1.11
- net PortExpander GPA4: no longer R9.8, U2.15
- net PortExpander GPB0: now also R13.8, U4.15; no longer R9.6, U2.11
- net PortExpander GPB1: now also R13.7, U4.13; no longer R9.5, U2.9
- net PortExpander GPB2: no longer R13.8, U4.15
- net PortExpander GPB3: no longer R13.7, U4.13
- new net GPIO 13 (PIN 15): R9.6, U2.11
- new net GPIO 14 (PIN 12): R9.5, U2.9
- new net GPIO 4 (PIN 26): R10.5, U1.9
