File: Hardware/KICAD/PortExpander.kicad_sch (KiCad schematic)
At the start: 6 parts, among them U501 MCP23017_ML

Commit message: Add files via upload
Parts:
- added K501, K502, K503, K504: K31, Connector_Wire:SolderWire-0.5sqmm_1x01_D0.9mm_OD2.1mm, symbol Connector_Generic:Conn_01x01
- U501: footprint Package_DFN_QFN:QFN-28-1EP_6x6mm_P0.65mm_EP4.25x4.25mm -> Package_SO:SSOP-28_5.3x10.2mm_P0.65mm; symbol Interface_Expansion:MCP23017_ML -> Interface_Expansion:MCP23017_SS
Connections:
- net 3,3 V from ESP: now also U501.9 (VDD); no longer U501.5 (VDD)
- net GND: now also U501.10 (VSS), U501.15 (A0), U501.16 (A1), U501.17 (A2); no longer U501.11 (A0), U501.12 (A1), U501.13 (A2), U501.6 (VSS)
- net GPIO 26 (PIN 10): now also U501.13 (SDA); no longer U501.9 (SDA)
- net GPIO 27 (PIN 11): now also U501.12 (SCK); no longer U501.8 (SCK)
- net GPIO 32 (PIN 7): now also U501.19 (INTB); no longer U501.15 (INTB)
- net GPIO 33 (PIN 8): now also U501.20 (INTA); no longer U501.16 (INTA)
- net PortExpander GPA0: now also U501.21 (GPA0); no longer U501.17 (GPA0)
- net PortExpander GPA1: now also U501.22 (GPA1); no longer U501.18 (GPA1)
- net PortExpander GPA2: now also U501.23 (GPA2); no longer U501.19 (GPA2)
- net PortExpander GPA3: now also U501.24 (GPA3); no longer U501.20 (GPA3)
- net PortExpander GPA4: now also U501.25 (GPA4); no longer U501.21 (GPA4)
- net PortExpander GPA5: now also U501.26 (GPA5); no longer U501.22 (GPA5)
- net PortExpander GPB0: now also U501.1 (GPB0); no longer U501.25 (GPB0)
- net PortExpander GPB1: now also U501.2 (GPB1); no longer U501.26 (GPB1)
- net PortExpander GPB2: now also U501.3 (GPB2); no longer U501.27 (GPB2)
- net PortExpander GPB3: now also U501.4 (GPB3); no longer U501.28 (GPB3)
- net PortExpander GPB4: now also U501.5 (GPB4); no longer U501.1 (GPB4)
- net PortExpander GPB5: now also U501.6 (GPB5); no longer U501.2 (GPB5)
- net at C502.2, R501.2: now also U501.18 (~{RESET}); no longer U501.14 (~{RESET})
- net GPB6: now reaches U501.7 (GPB6)
- net GPB6: now also K501.1 (Pin_1)
- new net GPA6: K503.1 (Pin_1), U501.27 (GPA6)
- new net GPA7: K504.1 (Pin_1), U501.28 (GPA7)
- new net GPB7: K502.1 (Pin_1), U501.8 (GPB7)
